Commit message: Added gazebo specific controller configuration and played with inertias

File: aero_description/urdf/husky.urdf.xacro (robot description, xacro)
@@ -53,9 +53,9 @@
       <inertial>
 	<origin xyz="0 0 0" rpy="0 0 0"/>
-	<mass value="1"/>
+	<mass value="5"/>
 	<inertia
 	    ixx="1.0" ixy="0.0" ixz="0.0"
-	    iyy="1.0" iyz="0.0"
-	    izz="1.0"/>
+	    iyy="0.0" iyz="0.0"
+	    izz="0.0"/>
       </inertial>
     </link>
