Commit message: Added static interface for eth-back

File: aero_description/urdf/camera_boom.urdf.xacro (robot description, xacro)
@@ -51,6 +51,6 @@
     </xacro:static_transform>
     <!-- Cameras -->
-    <xacro:stereo_camera_pair parent="${robot_ns}/boom_top" prefix="${robot_ns}/upper_stereo" xyz="0 0 0.005" rpy="0 0 0" camera_base_length="0.3" camera_tilt="${12*M_PI/180}"/>
-    <xacro:stereo_camera_pair parent="${robot_ns}/boom_top" prefix="${robot_ns}/lower_stereo" xyz="0 0 -0.127" rpy="0 0 0" camera_base_length="0.11" camera_tilt="${34*M_PI/180}"/>
+    <xacro:stereo_camera_pair parent="${robot_ns}/boom_top" prefix="${robot_ns}/upper_stereo" xyz="0 0 0.005" rpy="0 0 0" camera_base_length="0.3" camera_tilt="${12*M_PI/180}" stereo_optical_frame_offset="0.2"/>
+    <xacro:stereo_camera_pair parent="${robot_ns}/boom_top" prefix="${robot_ns}/lower_stereo" xyz="0 0 -0.127" rpy="0 0 0" camera_base_length="0.11" camera_tilt="${34*M_PI/180}" stereo_optical_frame_offset="0.1"/>
   </xacro:macro>
 </robot>

File: aero_description/urdf/stereo_camera_pair.urdf.xacro (robot description, xacro)
@@ -8,5 +8,5 @@
   <property name="camera_rail_length" value="0.0508" /><!--front to back -->
   <property name="camera_rail_height" value="0.0254" />
-  <xacro:macro name="stereo_camera_pair" params="prefix parent xyz rpy camera_base_length camera_tilt">
+  <xacro:macro name="stereo_camera_pair" params="prefix parent xyz rpy camera_base_length camera_tilt stereo_optical_frame_offset">
     <xacro:static_transform parent="${parent}" name="${prefix}/camera_rail" xyz="${xyz}" rpy="${rpy}">
     <visual>
@@ -60,5 +60,5 @@
       <origin xyz="0.03 ${-camera_base_length/2} ${manta_camera_height/2+camera_rail_height/2}" rpy="0 0 0" />
     </xacro:manta_cam_v0>
-    <xacro:static_transform parent="${prefix}/camera_rail_tilt" name="${prefix}/optical_frame" xyz="0.03 0 ${manta_camera_height/2+camera_rail_height/2}" rpy="${-M_PI/2} 0 ${-M_PI/2}">
+    <xacro:static_transform parent="${prefix}/camera_rail_tilt" name="${prefix}/optical_frame" xyz="${stereo_optical_frame_offset+0.04} 0 ${manta_camera_height/2+camera_rail_height/2}" rpy="${-M_PI/2} 0 ${-M_PI/2}">
       <visual>
 	<geometry>
