Commit message: Fixed wheels so there is nolonger a cyclic mimic

File: aero_description/urdf/base.urdf.xacro (robot description, xacro)
@@ -64,8 +64,9 @@
 	</visual>
 	<collision>
-	  <origin xyz="0 0 ${wheel_x_size/2 - base_z_origin_to_wheel_origin - 0.02}" rpy="0 0 0 " />
+	  <origin xyz="0 0 0" rpy="0 0 0" />
 	  <geometry>
-	    <box size = "${base_x_size+0.02} ${base_y_size} ${base_z_size + 0.02}"/> <!--making it slightly bigger in x and z direction-->
+	    <mesh filename="package://aero_description/meshes/base_collision.STL" />
 	  </geometry>
+	  <material name="Black" />
 	</collision>
       </link>
@@ -75,8 +76,8 @@
       </gazebo>
       <!-- WHEEL macros -->
-      <husky_wheel fb="back" lr="left" parent="${robot_ns}/base_link" translateX="-1" translateY="1" flipY="-1" robot_ns="${robot_ns}"/>
-      <husky_wheel fb="back" lr="right" parent="${robot_ns}/base_link" translateX="-1" translateY="-1" flipY="-1" robot_ns="${robot_ns}"/>
-      <husky_wheel fb="front" lr="left" parent="${robot_ns}/base_link" translateX="1" translateY="1" flipY="-1" robot_ns="${robot_ns}"/>
-      <husky_wheel fb="front" lr="right" parent="${robot_ns}/base_link" translateX="1" translateY="-1" flipY="-1" robot_ns="${robot_ns}"/>
+      <husky_wheel fb="back" lr="left" parent="${robot_ns}/base_link" translateX="-1" translateY="1" flipY="-1" robot_ns="${robot_ns}" mimic="true"/>
+      <husky_wheel fb="back" lr="right" parent="${robot_ns}/base_link" translateX="-1" translateY="-1" flipY="-1" robot_ns="${robot_ns}" mimic="true"/>
+      <husky_wheel fb="front" lr="left" parent="${robot_ns}/base_link" translateX="1" translateY="1" flipY="-1" robot_ns="${robot_ns}" mimic="false"/>
+      <husky_wheel fb="front" lr="right" parent="${robot_ns}/base_link" translateX="1" translateY="-1" flipY="-1" robot_ns="${robot_ns}" mimic="false"/>
       <!-- DECORATIONS -->
       <!-- Top Plate -->

File: aero_description/urdf/wheel.urdf.xacro (robot description, xacro)
@@ -19,5 +19,5 @@
 	<property name="base_y_origin_to_wheel_origin" value="0.285475" />
 	<property name="base_z_origin_to_wheel_origin" value="0.03282508" />
-	<xacro:macro name="husky_wheel" params="fb lr parent translateX translateY flipY robot_ns"> <!--fb : front, back ; lr: left, right -->
+	<xacro:macro name="husky_wheel" params="fb lr parent translateX translateY flipY robot_ns mimic"> <!--fb : front, back ; lr: left, right -->
 		<link name="${robot_ns}/${fb}_${lr}_wheel">
 			<inertial>
@@ -57,5 +57,7 @@
 			<limit effort="100" velocity="100"/>
 			<joint_properties damping="0.0" friction="0.0"/>
-			<mimic joint="${robot_ns}/joint_front_${lr}_wheel" multiplier="1.0" offset="0.0" />
+			<xacro:if value="${mimic}">
+				<mimic joint="${robot_ns}/joint_front_${lr}_wheel" multiplier="1.0" offset="0.0" />
+			</xacro:if>
 		</joint>
 		<transmission name="${robot_ns}/${fb}_${lr}_wheel_tran">

Commit message: Added base_collision in Collada format and reinitialized with MoveIt wizard

File: aero_description/urdf/base.urdf.xacro (robot description, xacro)
@@ -66,5 +66,5 @@
 	  <origin xyz="-0.40 -0.203 0" rpy="${M_PI/2} 0 ${M_PI/2}" />
 	  <geometry>
-            <mesh filename="package://aero_description/meshes/base_collision.STL" />
+            <mesh filename="package://aero_description/meshes/base_collision.dae" />
 	  </geometry>
 	  <material name="Black" />
