Commit message: Removed camera collision model

File: aero_description/urdf/manta_camera.urdf.xacro (robot description, xacro)
@@ -4,5 +4,5 @@
       xmlns:interface="http://playerstage.sourceforge.net/gazebo/xmlschema/#interface"
       xmlns:xacro="http://ros.org/wiki/xacro">
-  <xacro:include filename="$(find aero_description)/urdf/manta_camera.gazebo.xacro" />
+  <!--<xacro:include filename="$(find aero_description)/urdf/manta_camera.gazebo.xacro" />-->
   <property name="manta_camera_width" value="0.04" />
   <property name="manta_camera_height" value="0.02" />
@@ -27,10 +27,4 @@
                  izz="0.001" />
       </inertial>
-     <collision>
-      <origin xyz="0 0 0" rpy="0 0 0" />
-      <geometry>
-        <mesh filename="package://aero_description/meshes/Manta-Camera-Lense.STL" />
-      </geometry>
-    </collision>
     </link>
     <joint name="${frame_name}_optical_frame_joint" type="fixed">
