Commit message: Added laser scanner to model Switched to asphalt ground in world Made robot heavier

File: aero_description/robots/aero_base.urdf.xacro (robot description, xacro)
@@ -8,7 +8,7 @@
   <xacro:husky/>
   <!-- Laser -->
-  <!--<xacro:sick_laser_v0 name="laser" parent="base_link" ros_topic="laser" update_rate="25" >
-    <origin xyz="${base_length/2+0.0635} 0 0.0254" rpy="${M_PI} 0 0" />
-  </xacro:sick_laser_v0>-->
+  <xacro:sick_laser_v0 name="laser" parent="base_link" ros_topic="laser" update_rate="25" >
+    <origin xyz="${base_x_size/2+0.0635} 0 0.0254" rpy="${M_PI} 0 0" />
+  </xacro:sick_laser_v0>
   <!-- IMU -->
   <xacro:static_transform parent="base_link" name="imu" xyz="0 0 0" rpy="0 ${-M_PI/2} ${-3*M_PI/4}">

File: aero_description/urdf/base.urdf.xacro (robot description, xacro)
@@ -18,5 +18,5 @@
     <property name="base_z_size" value="0.24750000" />
     <!--Weight of the base-->
-    <property name="base_mass" value="33.45489000" /> <!-- in kg-->
+    <property name="base_mass" value="70.45489000" /> <!-- in kg-->
     <!--Inertial values for the base at center of mass, aligned with coordinate system. Units are kg*m^2-->
     <property name="base_ixx_com_cs" value="0.60216370" />

File: aero_description/urdf/sick_laser.gazebo.xacro (robot description, xacro)
@@ -3,31 +3,32 @@
   <xacro:macro name="sick_laser_gazebo_v0" params="name ros_topic update_rate">
     <gazebo reference="${name}_link">
-      <sensor type="ray" name="${name}">
-        <always_on>true</always_on>
-        <update_rate>${update_rate}</update_rate>
-        <pose>0 0 0 0 0 0</pose>
-        <visualize>true</visualize>
-        <ray>
-          <scan>
-            <horizontal>
-              <samples>640</samples>
-              <resolution>1</resolution>
-              <min_angle>-135</min_angle>
-              <max_angle>135</max_angle>
-            </horizontal>
-          </scan>
-          <range>
-            <min>0.5</min>
-            <max>50.0</max>
-            <resolution>${0.25*180.0/M_PI}</resolution>
-          </range>
-        </ray>
-        <plugin name="gazebo_ros_${name}_controller" filename="libgazebo_ros_laser.so">
-          <gaussianNoise>0.005</gaussianNoise>
-          <alwaysOn>true</alwaysOn>
-          <updateRate>${update_rate}</updateRate>
-          <topicName>${ros_topic}</topicName>
-          <frameName>${name}_link</frameName>
-        </plugin>
+      <sensor type="ray" name="${name}_sensor">
+	<pose>0 0 0 0 0 0</pose>
+	<visualize>false</visualize>
+	<update_rate>${update_rate}</update_rate>
+	<ray>
+	  <scan>
+	    <horizontal>
+	      <samples>640</samples>
+	      <resolution>1</resolution>
+	      <min_angle>-2.35619</min_angle>
+	      <max_angle>2.35619</max_angle>
+	    </horizontal>
+	  </scan>
+	  <range>
+	    <min>0.5</min>
+	    <max>50.0</max>
+	    <resolution>0.01</resolution>
+	  </range>
+	  <noise>
+	    <type>gaussian</type>
+	    <mean>0.0</mean>
+	    <stddev>0.01</stddev>
+	  </noise>
+	</ray>
+	<plugin name="gazebo_ros_head_hokuyo_controller" filename="libgazebo_ros_laser.so">
+	  <topicName>${ros_topic}</topicName>
+	  <frameName>${name}_link</frameName>
+	</plugin>
       </sensor>
     </gazebo>

File: aero_description/urdf/sick_laser.urdf.xacro (robot description, xacro)
@@ -7,7 +7,7 @@
       <insert_block name="origin" />
       <parent link="${parent}"/>
-      <child link="${name}"/>
+      <child link="${name}_link"/>
     </joint>
-    <link name="${name}" type="laser">
+    <link name="${name}_link">
       <inertial>
         <mass value="0.001" />

File: aero_description/urdf/wheel.urdf.xacro (robot description, xacro)
@@ -39,9 +39,18 @@
 				    <cylinder length="${wheel_z_size}" radius="${wheel_x_size/2}" />
 				</geometry>
+				<surface>
+				  <friction>
+				    <ode mu='100.000000' mu2='100.000000' fdir1='0.000000 0.000000 0.000000' slip1='0.000000' slip2='0.000000'/>
+				  </friction>
+				  <bounce restitution_coefficient='0.000000' threshold='100000.000000'/>
+				  <contact>
+				    <ode soft_cfm='0.000000' soft_erp='0.200000' kp='1000000.000000' kd='1.000000' max_vel='100.000000' min_depth='0.000000'/>
+				  </contact>
+				</surface>
 			</collision>
 		</link>
 		<gazebo reference="${fb}_${lr}_wheel">
-			<mu1 value="1.0"/>
-			<mu2 value="1.0"/>
+			<mu1 value="0.4"/>
+			<mu2 value="0.4"/>
 			<kp  value="10000000.0" />
 			<kd  value="1.0" />

Commit message: Added stereo cameras to simulator

File: aero_description/robots/aero_base.urdf.xacro (robot description, xacro)
@@ -6,4 +6,5 @@
   <xacro:include filename="$(find aero_description)/urdf/sick_laser.urdf.xacro" />
   <xacro:include filename="$(find aero_description)/urdf/simple_transform.urdf.xacro" />
+  <xacro:include filename="$(find aero_description)/urdf/camera_boom.urdf.xacro" />
   <xacro:husky/>
   <!-- Laser -->
@@ -11,4 +12,29 @@
     <origin xyz="${base_x_size/2+0.0635} 0 0.0254" rpy="${M_PI} 0 0" />
   </xacro:sick_laser_v0>
+  <!-- Camera Boom -->
+  <xacro:aero_camera_boom boom_base="aero_boom_base"/>
+  <xacro:static_transform parent="base_footprint" name="aero_boom_base" xyz="-0.4191 0 0.28575" rpy="0 0 0">
+    <visual>
+      <origin xyz="0 0 -0.02" rpy="0 0 0" />
+      <geometry>
+	<box size="0.05 0.05 0.05" />
+      </geometry>
+      <material name="Blue" />
+    </visual>
+    <collision>
+      <origin xyz="0 0 -0.02" rpy="0 0 0" />
+      <geometry>
+	<box size="0.05 0.05 0.05" />
+      </geometry>
+    </collision>
+    <inertial>
+      <origin xyz="0 0 0" rpy="0 0 0"/>
+      <mass value="1"/>
+      <inertia
+	  ixx="1.0" ixy="0.0" ixz="0.0"
+	  iyy="1.0" iyz="0.0"
+	  izz="1.0"/>
+    </inertial>
+  </xacro:static_transform>
   <!-- IMU -->
   <xacro:static_transform parent="base_link" name="imu" xyz="0 0 0" rpy="0 ${-M_PI/2} ${-3*M_PI/4}">

File: aero_description/urdf/manta_camera.urdf.xacro (robot description, xacro)
@@ -49,5 +49,5 @@
     </link>
     <!-- extensions -->
-    <xacro:manta_cam_gazebo_v0 camera_name="${camera_name}" frame_name="${frame_name}" />
+    <!--<xacro:manta_cam_gazebo_v0 camera_name="${camera_name}" frame_name="${frame_name}" />-->
   </xacro:macro>
 </root>

File: aero_description/urdf/stereo_camera_pair.urdf.xacro (robot description, xacro)
@@ -17,4 +17,18 @@
       <material name="Blue"/>
     </visual>
+    <collision>
+      <origin xyz="0 0 ${camera_rail_height/2}" rpy="0 0 0" />
+      <geometry>
+	<box size="${camera_rail_length} ${camera_base_length-manta_camera_width} ${camera_rail_height}" />
+      </geometry>
+    </collision>
+    <inertial>
+      <origin xyz="0 0 0" rpy="0 0 0"/>
+      <mass value="1"/>
+      <inertia
+	  ixx="1.0" ixy="0.0" ixz="0.0"
+	  iyy="1.0" iyz="0.0"
+	  izz="1.0"/>
+    </inertial>
   </xacro:static_transform>
   <xacro:static_transform parent="${prefix}/camera_rail" name="${prefix}/camera_rail_tilt" xyz="0 0 ${camera_rail_height/2}" rpy="0 ${camera_tilt} 0">
@@ -25,4 +39,18 @@
       </geometry>
     </visual>
+    <collision>
+      <origin xyz="0 0 0" rpy="0 0 0" />
+      <geometry>
+	<box size="0 0 0" />
+      </geometry>
+    </collision>
+    <inertial>
+      <origin xyz="0 0 0" rpy="0 0 0"/>
+      <mass value="1"/>
+      <inertia
+	  ixx="1.0" ixy="0.0" ixz="0.0"
+	  iyy="1.0" iyz="0.0"
+	  izz="1.0"/>
+    </inertial>
   </xacro:static_transform>
     <xacro:manta_cam_v0 frame_name="${prefix}/left_camera" parent="${prefix}/camera_rail_tilt" camera_name="${prefix}/left">
@@ -32,14 +60,82 @@
       <origin xyz="0.03 ${-camera_base_length/2} ${manta_camera_height/2+camera_rail_height/2}" rpy="0 0 0" />
     </xacro:manta_cam_v0>
-    <xacro:static_transform parent="${prefix}/camera_rail_tilt" name="${prefix}_optical_frame" xyz="0.03 0 ${manta_camera_height/2+camera_rail_height/2}" rpy="${-M_PI/2} 0 ${-M_PI/2}">
-    <visual>
-      <geometry>
-	<box size="0 0 0" />
-      </geometry>
-      <material name="Clear">
-	<color rgba="0 0 0 0"/>
-      </material>
-    </visual>
-  </xacro:static_transform>
+    <xacro:static_transform parent="${prefix}/camera_rail_tilt" name="${prefix}/optical_frame" xyz="0.03 0 ${manta_camera_height/2+camera_rail_height/2}" rpy="${-M_PI/2} 0 ${-M_PI/2}">
+      <visual>
+	<geometry>
+	  <box size="0 0 0" />
+	</geometry>
+	<material name="Clear">
+	  <color rgba="0 0 0 0"/>
+	</material>
+      </visual>
+      <collision>
+	<geometry>
+	  <box size="0 0 0" />
+	</geometry>
+      </collision>
+      <inertial>
+	<origin xyz="0 0 0" rpy="0 0 0"/>
+	<mass value="1"/>
+	<inertia
+	    ixx="1.0" ixy="0.0" ixz="0.0"
+	    iyy="1.0" iyz="0.0"
+	    izz="1.0"/>
+      </inertial>
+    </xacro:static_transform>
+    <gazebo reference="${prefix}/camera_rail_tilt">
+      <sensor type="multicamera" name="${prefix}/camera">
+	<update_rate>30.0</update_rate>
+	<camera name="left">
+	  <pose>0.1 ${camera_base_length/2} ${manta_camera_height/2+camera_rail_height/2} 0 0 0</pose>
+	  <horizontal_fov>1.3962634</horizontal_fov>
+	  <image>
+	    <width>800</width>
+	    <height>800</height>
+	    <format>R8G8B8</format>
+	  </image>
+	  <clip>
+	    <near>0.02</near>
+	    <far>300</far>
+	  </clip>
+	  <noise>
+	    <type>gaussian</type>
+	    <mean>0.0</mean>
+	    <stddev>0.007</stddev>
+	  </noise>
+	</camera>
+	<camera name="right">
+	  <pose>0.1 ${-camera_base_length/2} ${manta_camera_height/2+camera_rail_height/2} 0 0 0</pose>
+	  <horizontal_fov>1.3962634</horizontal_fov>
+	  <image>
+	    <width>800</width>
+	    <height>800</height>
+	    <format>R8G8B8</format>
+	  </image>
+	  <clip>
+	    <near>0.02</near>
+	    <far>300</far>
+	  </clip>
+	  <noise>
+	    <type>gaussian</type>
+	    <mean>0.0</mean>
+	    <stddev>0.007</stddev>
+	  </noise>
+	</camera>
+	<plugin name="${prefix}/camera_controller" filename="libgazebo_ros_multicamera.so">
+	  <alwaysOn>true</alwaysOn>
+	  <updateRate>0.0</updateRate>
+	  <cameraName>${prefix}/camera</cameraName>
+	  <imageTopicName>image_raw</imageTopicName>
+	  <cameraInfoTopicName>camera_info</cameraInfoTopicName>
+	  <frameName>${prefix}/optical_frame</frameName>
+	  <hackBaseline>0.07</hackBaseline>
+	  <distortionK1>0.0</distortionK1>
+	  <distortionK2>0.0</distortionK2>
+	  <distortionK3>0.0</distortionK3>
+	  <distortionT1>0.0</distortionT1>
+	  <distortionT2>0.0</distortionT2>
+	</plugin>
+      </sensor>
+    </gazebo>
   </xacro:macro>
 </root>

Commit message: Added namespaces to some frames and topics Added joint state publisher for boom joint

File: aero_description/robots/aero_base.urdf.xacro (robot description, xacro)
@@ -7,12 +7,13 @@
   <xacro:include filename="$(find aero_description)/urdf/simple_transform.urdf.xacro" />
   <xacro:include filename="$(find aero_description)/urdf/camera_boom.urdf.xacro" />
+  <property name="robot_ns" value="/aero" />
   <xacro:husky/>
   <!-- Laser -->
-  <xacro:sick_laser_v0 name="laser" parent="base_link" ros_topic="aero/laser" update_rate="25" >
+  <xacro:sick_laser_v0 name="laser" parent="base_link" ros_topic="${robot_ns}/laser" update_rate="25" >
     <origin xyz="${base_x_size/2+0.0635} 0 0.0254" rpy="${M_PI} 0 0" />
   </xacro:sick_laser_v0>
   <!-- Camera Boom -->
-  <xacro:aero_camera_boom boom_base="aero_boom_base"/>
-  <xacro:static_transform parent="base_footprint" name="aero_boom_base" xyz="-0.4191 0 0.28575" rpy="0 0 0">
+  <xacro:aero_camera_boom boom_base="${robot_ns}/boom_base" robot_ns="${robot_ns}"/>
+  <xacro:static_transform parent="base_footprint" name="${robot_ns}/boom_base" xyz="-0.4191 0 0.28575" rpy="0 0 0">
     <visual>
       <origin xyz="0 0 -0.02" rpy="0 0 0" />

File: aero_description/urdf/camera_boom.urdf.xacro (robot description, xacro)
@@ -3,7 +3,7 @@
   <property name="boom_length" value="1.085" />
   <property name="boom_diameter" value="0.0538" />
-  <xacro:macro name="aero_camera_boom" params="boom_base">
+  <xacro:macro name="aero_camera_boom" params="boom_base robot_ns">
     <!-- Boom -->
-    <xacro:revolute_pan_transform parent="${boom_base}" name="boom" xyz="0 0 0" rpy="0 0 0" lower_limit="-2" upper_limit="2">
+    <xacro:revolute_pan_transform parent="${boom_base}" name="${robot_ns}/boom" xyz="0 0 0" rpy="0 0 0" lower_limit="-2" upper_limit="2">
       <visual>
 	<origin xyz="0.0 0.0 ${boom_length/2}" rpy="0 0 0" />
@@ -28,5 +28,5 @@
       </inertial>
     </xacro:revolute_pan_transform>
-    <xacro:static_transform parent="boom" name="boom_top" xyz="0 0 ${boom_length}" rpy="0 0 0">
+    <xacro:static_transform parent="${robot_ns}/boom" name="${robot_ns}/boom_top" xyz="0 0 ${boom_length}" rpy="0 0 0">
       <visual>
 	<origin xyz="0 0 0" rpy="0 0 0" />
@@ -51,6 +51,6 @@
     </xacro:static_transform>
     <!-- Cameras -->
-    <xacro:stereo_camera_pair parent="boom_top" prefix="upper_stereo" xyz="0 0 0.005" rpy="0 0 0" camera_base_length="0.3" camera_tilt="${12*M_PI/180}"/>
-    <xacro:stereo_camera_pair parent="boom_top" prefix="lower_stereo" xyz="0 0 -0.127" rpy="0 0 0" camera_base_length="0.11" camera_tilt="${34*M_PI/180}"/>
+    <xacro:stereo_camera_pair parent="${robot_ns}/boom_top" prefix="${robot_ns}/upper_stereo" xyz="0 0 0.005" rpy="0 0 0" camera_base_length="0.3" camera_tilt="${12*M_PI/180}"/>
+    <xacro:stereo_camera_pair parent="${robot_ns}/boom_top" prefix="${robot_ns}/lower_stereo" xyz="0 0 -0.127" rpy="0 0 0" camera_base_length="0.11" camera_tilt="${34*M_PI/180}"/>
   </xacro:macro>
 </robot>
