Commit message: Added IMU to simulator Updated tf frames to start with aero prefix

File: aero_description/robots/aero_base.urdf.xacro (robot description, xacro)
@@ -8,12 +8,12 @@
   <xacro:include filename="$(find aero_description)/urdf/camera_boom.urdf.xacro" />
   <property name="robot_ns" value="/aero" />
-  <xacro:husky/>
+  <xacro:husky robot_ns="${robot_ns}"/>
   <!-- Laser -->
-  <xacro:sick_laser_v0 name="laser" parent="base_link" ros_topic="${robot_ns}/laser" update_rate="25" >
+  <xacro:sick_laser_v0 name="${robot_ns}/laser" parent="${robot_ns}/base_link" ros_topic="${robot_ns}/laser" update_rate="25" >
     <origin xyz="${base_x_size/2+0.0635} 0 0.0254" rpy="${M_PI} 0 0" />
   </xacro:sick_laser_v0>
   <!-- Camera Boom -->
   <xacro:aero_camera_boom boom_base="${robot_ns}/boom_base" robot_ns="${robot_ns}"/>
-  <xacro:static_transform parent="base_footprint" name="${robot_ns}/boom_base" xyz="-0.4191 0 0.28575" rpy="0 0 0">
+  <xacro:static_transform parent="${robot_ns}/base_footprint" name="${robot_ns}/boom_base" xyz="-0.4191 0 0.28575" rpy="0 0 0">
     <visual>
       <origin xyz="0 0 -0.02" rpy="0 0 0" />
@@ -39,5 +39,5 @@
   </xacro:static_transform>
   <!-- IMU -->
-  <xacro:static_transform parent="base_link" name="imu" xyz="0 0 0" rpy="0 ${-M_PI/2} ${-3*M_PI/4}">
+  <xacro:static_transform parent="${robot_ns}/base_link" name="${robot_ns}/imu" xyz="0 0 0" rpy="0 ${-M_PI/2} ${-3*M_PI/4}">
     <collision>
       <origin xyz="0 0 0" rpy="0 0 0" />
@@ -62,3 +62,50 @@
     </inertial>
   </xacro:static_transform>
+  <gazebo reference="${robot_ns}/imu">
+    <sensor name="imu_sensor" type="imu"><!--from atlas-->
+      <always_on>1</always_on>
+      <update_rate>1000.0</update_rate>
+      <imu>
+	<noise>
+	  <type>gaussian</type>
+	  <!-- Noise parameters from Boston Dynamics
+	       (http://gazebosim.org/wiki/Sensor_noise):
+	       rates (rad/s): mean=0, stddev=2e-4
+	       accels (m/s/s): mean=0, stddev=1.7e-2
+	       rate bias (rad/s): 5e-6 - 1e-5
+	       accel bias (m/s/s): 1e-1
+	       Experimentally, simulation provide rates with noise of
+	       about 1e-3 rad/s and accels with noise of about 1e-1 m/s/s.
+	       So we don't expect to see the noise unless number of inner iterations
+	       are increased.
+We will add bias.  In this model, bias is sampled once for rates
+and once for accels at startup; the sign (negative or positive)
+of each bias is then switched with equal probability.  Thereafter,
+the biases are fixed additive offsets.  We choose
+bias means and stddevs to produce biases close to the provided
+data. -->
+	  <rate>
+	    <mean>0.0</mean>
+	    <stddev>2e-4</stddev>
+	    <bias_mean>0.0000075</bias_mean>
+	    <bias_stddev>0.0000008</bias_stddev>
+	  </rate>
+	  <accel>
+	    <mean>0.0</mean>
+	    <stddev>1.7e-2</stddev>
+	    <bias_mean>0.1</bias_mean>
+	    <bias_stddev>0.001</bias_stddev>
+	  </accel>
+	</noise>
+      </imu>
+    </sensor>
+  </gazebo>
+  <gazebo><!-- need to put it in it's own gazebo tag with no reference because the imu plugin is a model plugin -->
+    <plugin filename="libgazebo_ros_imu.so" name="imu_controller">
+      <bodyName>${robot_ns}/imu</bodyName>
+      <robotNamespace>${robot_ns}</robotNamespace>
+      <topicName>imu</topicName>
+      <serviceName>imu/calibrate</serviceName>
+    </plugin>
+  </gazebo>
 </robot>

File: aero_description/urdf/base.urdf.xacro (robot description, xacro)
@@ -26,94 +26,96 @@
     <property name="base_iyz_com_cs" value="-0.00154437" />
     <property name="base_izz_com_cs" value="2.02955229" />
-<!-- BASE-FOOTPRINT -->
-    <!-- base_footprint is a fictitious link(frame) that is on the ground right below base_link origin, navigation stack depends on this frame -->
-    <link name="base_footprint">
-        <inertial>
-            <mass value="0.0001" />
-            <origin xyz="0 0 0" />
-            <inertia ixx="0.0001" ixy="0.0" ixz="0.0"
-                iyy="0.0001" iyz="0.0"
-                izz="0.0001" />
-        </inertial>
-        <visual>
-            <origin xyz="0 0 0" rpy="0 0 0" />
-            <geometry>
-                <box size="0.001 0.001 0.001" />
-            </geometry>
-        </visual>
-    </link>
-    <gazebo reference="base_footprint">
-        <turnGravityOff>false</turnGravityOff>
-    </gazebo>
-    <joint name="base_footprint_joint" type="fixed">
-		<origin xyz="0 0 ${wheel_x_size/2 - base_z_origin_to_wheel_origin}" rpy="0 0 0" />
-        <parent link="base_footprint"/>
-        <child link="base_link" />
-    </joint>
-    <!-- BASE-LINK -->
-    <!--Actual body/chassis of the robot-->
-    <link name="base_link">
-        <inertial>
-            <mass value="${base_mass}" />
-            <!--This is the pose of the inertial reference frame, relative to the link reference frame. The origin of the inertial reference frame needs to be at the center of gravity. The axes of the inertial reference frame do not need to be aligned with the principal axes of the inertia.-->
-            <origin xyz="${base_x_com} ${base_y_com} ${base_z_com}" />
-            <!--The 3x3 rotational inertia matrix. Because the rotational inertia matrix is symmetric, only 6 above-diagonal elements of this matrix are specified here, using the attributes ixx, ixy, ixz, iyy, iyz, izz.-->
-            <inertia ixx="${base_ixx_com_cs}" ixy="${base_ixy_com_cs}" ixz="${base_ixz_com_cs}"
-                iyy="${base_iyy_com_cs}" iyz="${base_iyz_com_cs}" izz="${base_izz_com_cs}" />
-        </inertial>
-        <visual>
-            <origin xyz="0 0 0" rpy="0 0 0" />
-            <geometry>
-                <mesh filename="package://husky_description/meshes/base_link.stl" />
-            </geometry>
-            <material name="Black" />
-        </visual>
-		<collision>
-			<origin xyz="0 0 ${wheel_x_size/2 - base_z_origin_to_wheel_origin - 0.02}" rpy="0 0 0 " />
-			<geometry>
-				<box size = "${base_x_size+0.02} ${base_y_size} ${base_z_size + 0.02}"/> <!--making it slightly bigger in x and z direction-->
-			</geometry>
-		</collision>
-    </link>
-    <gazebo reference="base_link">
-        <material>Gazebo/FlatBlack</material>
-        <turnGravityOff>false</turnGravityOff>
-    </gazebo>
-    <!-- WHEEL macros -->
-	<husky_wheel fb="back" lr="left" parent="base_link" translateX="-1" translateY="1" flipY="-1"/>
-	<husky_wheel fb="back" lr="right" parent="base_link" translateX="-1" translateY="-1" flipY="-1"/>
-	<husky_wheel fb="front" lr="left" parent="base_link" translateX="1" translateY="1" flipY="-1"/>
-	<husky_wheel fb="front" lr="right" parent="base_link" translateX="1" translateY="-1" flipY="-1"/>
-    <!-- DECORATIONS -->
-    <!-- Top Plate -->
-    <husky_part parent="base_footprint" name="top_plate" mesh="top_plate"
-          colour="Yellow"
-          translateX="0.0" translateY="0.0" translateZ="${wheel_x_size/2 - base_z_origin_to_wheel_origin}"
-          rotateX="0.0" rotateY="0.0" rotateZ="0.0"/>
-    <gazebo reference="base_footprint_top_plate_part">
-        <material>Gazebo/Yellow</material>
-    </gazebo>
-    <!-- User Rail -->
-    <husky_part parent="base_footprint" name="user_rail" mesh="user_rail"
-          colour="DarkGray"
-          translateX="0.272" translateY="0.0" translateZ="${0.245 + wheel_x_size/2 - base_z_origin_to_wheel_origin}"
-          rotateX="0.0" rotateY="0.0" rotateZ="0.0"/>
-    <gazebo reference="base_footprint_user_rail_part">
-        <material>Gazebo/Grey</material>
-    </gazebo>
-    <!-- Bumpers -->
-    <husky_part parent="base_footprint" name="front_bumper" mesh="bumper"
-          colour="DarkGray"
-          translateX="0.490" translateY="0.0" translateZ="${0.091 + wheel_x_size/2 - base_z_origin_to_wheel_origin}"
-          rotateX="0.0" rotateY="0.0" rotateZ="0.0"/>
-    <gazebo reference="base_footprint_front_bumper_part">
-        <material>Gazebo/FlatBlack</material>
-    </gazebo>
-    <husky_part parent="base_footprint" name="rear_bumper" mesh="bumper"
-          colour="DarkGray"
-          translateX="-0.48" translateY="0.0" translateZ="${0.091 + wheel_x_size/2 - base_z_origin_to_wheel_origin}"
-          rotateX="0.0" rotateY="0.0" rotateZ="3.14"/>
-    <gazebo reference="base_footprint_rear_bumper_part">
-        <material>Gazebo/FlatBlack</material>
-    </gazebo>
+    <xacro:macro name="husky" params="robot_ns">
+      <!-- BASE-FOOTPRINT -->
+      <!-- base_footprint is a fictitious link(frame) that is on the ground right below base_link origin, navigation stack depends on this frame -->
+      <link name="${robot_ns}/base_footprint">
+	<inertial>
+	  <mass value="0.0001" />
+	  <origin xyz="0 0 0" />
+	  <inertia ixx="0.0001" ixy="0.0" ixz="0.0"
+		   iyy="0.0001" iyz="0.0"
+		   izz="0.0001" />
+	</inertial>
+	<visual>
+	  <origin xyz="0 0 0" rpy="0 0 0" />
+	  <geometry>
+	    <box size="0.001 0.001 0.001" />
+	  </geometry>
+	</visual>
+      </link>
+      <gazebo reference="${robot_ns}/base_footprint">
+	<turnGravityOff>false</turnGravityOff>
+      </gazebo>
+      <joint name="${robot_ns}/base_footprint_joint" type="fixed">
+	<origin xyz="0 0 ${wheel_x_size/2 - base_z_origin_to_wheel_origin}" rpy="0 0 0" />
+	<parent link="${robot_ns}/base_footprint"/>
+	<child link="${robot_ns}/base_link" />
+      </joint>
+      <!-- BASE-LINK -->
+      <!--Actual body/chassis of the robot-->
+      <link name="${robot_ns}/base_link">
+	<inertial>
+	  <mass value="${base_mass}" />
+	  <!--This is the pose of the inertial reference frame, relative to the link reference frame. The origin of the inertial reference frame needs to be at the center of gravity. The axes of the inertial reference frame do not need to be aligned with the principal axes of the inertia.-->
+	  <origin xyz="${base_x_com} ${base_y_com} ${base_z_com}" />
+	  <!--The 3x3 rotational inertia matrix. Because the rotational inertia matrix is symmetric, only 6 above-diagonal elements of this matrix are specified here, using the attributes ixx, ixy, ixz, iyy, iyz, izz.-->
+	  <inertia ixx="${base_ixx_com_cs}" ixy="${base_ixy_com_cs}" ixz="${base_ixz_com_cs}"
+		   iyy="${base_iyy_com_cs}" iyz="${base_iyz_com_cs}" izz="${base_izz_com_cs}" />
+	</inertial>
+	<visual>
+	  <origin xyz="0 0 0" rpy="0 0 0" />
+	  <geometry>
+	    <mesh filename="package://husky_description/meshes/base_link.stl" />
+	  </geometry>
+	  <material name="Black" />
+	</visual>
+	<collision>
+	  <origin xyz="0 0 ${wheel_x_size/2 - base_z_origin_to_wheel_origin - 0.02}" rpy="0 0 0 " />
+	  <geometry>
+	    <box size = "${base_x_size+0.02} ${base_y_size} ${base_z_size + 0.02}"/> <!--making it slightly bigger in x and z direction-->
+	  </geometry>
+	</collision>
+      </link>
+      <gazebo reference="${robot_ns}/base_link">
+	<material>Gazebo/FlatBlack</material>
+	<turnGravityOff>false</turnGravityOff>
+      </gazebo>
+      <!-- WHEEL macros -->
+      <husky_wheel fb="back" lr="left" parent="${robot_ns}/base_link" translateX="-1" translateY="1" flipY="-1" robot_ns="${robot_ns}"/>
+      <husky_wheel fb="back" lr="right" parent="${robot_ns}/base_link" translateX="-1" translateY="-1" flipY="-1" robot_ns="${robot_ns}"/>
+      <husky_wheel fb="front" lr="left" parent="${robot_ns}/base_link" translateX="1" translateY="1" flipY="-1" robot_ns="${robot_ns}"/>
+      <husky_wheel fb="front" lr="right" parent="${robot_ns}/base_link" translateX="1" translateY="-1" flipY="-1" robot_ns="${robot_ns}"/>
+      <!-- DECORATIONS -->
+      <!-- Top Plate -->
+      <husky_part parent="${robot_ns}/base_footprint" name="top_plate" mesh="top_plate"
+		  colour="Yellow"
+		  translateX="0.0" translateY="0.0" translateZ="${wheel_x_size/2 - base_z_origin_to_wheel_origin}"
+		  rotateX="0.0" rotateY="0.0" rotateZ="0.0"/>
+      <gazebo reference="${robot_ns}/base_footprint_top_plate_part">
+	<material>Gazebo/Yellow</material>
+      </gazebo>
+      <!-- User Rail -->
+      <husky_part parent="${robot_ns}/base_footprint" name="user_rail" mesh="user_rail"
+		  colour="DarkGray"
+		  translateX="0.272" translateY="0.0" translateZ="${0.245 + wheel_x_size/2 - base_z_origin_to_wheel_origin}"
+		  rotateX="0.0" rotateY="0.0" rotateZ="0.0"/>
+      <gazebo reference="base_footprint_user_rail_part">
+	<material>Gazebo/Grey</material>
+      </gazebo>
+      <!-- Bumpers -->
+      <husky_part parent="${robot_ns}/base_footprint" name="front_bumper" mesh="bumper"
+		  colour="DarkGray"
+		  translateX="0.490" translateY="0.0" translateZ="${0.091 + wheel_x_size/2 - base_z_origin_to_wheel_origin}"
+		  rotateX="0.0" rotateY="0.0" rotateZ="0.0"/>
+      <gazebo reference="${robot_ns}/base_footprint_front_bumper_part">
+	<material>Gazebo/FlatBlack</material>
+      </gazebo>
+      <husky_part parent="${robot_ns}/base_footprint" name="rear_bumper" mesh="bumper"
+		  colour="DarkGray"
+		  translateX="-0.48" translateY="0.0" translateZ="${0.091 + wheel_x_size/2 - base_z_origin_to_wheel_origin}"
+		  rotateX="0.0" rotateY="0.0" rotateZ="3.14"/>
+      <gazebo reference="${robot_ns}/base_footprint_rear_bumper_part">
+	<material>Gazebo/FlatBlack</material>
+      </gazebo>
+    </xacro:macro>
 </robot>

File: aero_description/urdf/wheel.urdf.xacro (robot description, xacro)
@@ -19,6 +19,6 @@
 	<property name="base_y_origin_to_wheel_origin" value="0.285475" />
 	<property name="base_z_origin_to_wheel_origin" value="0.03282508" />
-	<xacro:macro name="husky_wheel" params="fb lr parent translateX translateY flipY"> <!--fb : front, back ; lr: left, right -->
-		<link name="${fb}_${lr}_wheel">
+	<xacro:macro name="husky_wheel" params="fb lr parent translateX translateY flipY robot_ns"> <!--fb : front, back ; lr: left, right -->
+		<link name="${robot_ns}/${fb}_${lr}_wheel">
 			<inertial>
 				<mass value="${wheel_mass}" />
@@ -41,5 +41,5 @@
 			</collision>
 		</link>
-		<gazebo reference="${fb}_${lr}_wheel">
+		<gazebo reference="${robot_ns}/${fb}_${lr}_wheel">
 			<mu1 value="0.4"/>
 			<mu2 value="0.4"/>
@@ -50,7 +50,7 @@
 			<turnGravityOff>false</turnGravityOff>
 		</gazebo>
-		<joint name="joint_${fb}_${lr}_wheel" type="continuous">
+		<joint name="${robot_ns}/joint_${fb}_${lr}_wheel" type="continuous">
 			<parent link="${parent}"/>
-			<child link="${fb}_${lr}_wheel"/>
+			<child link="${robot_ns}/${fb}_${lr}_wheel"/>
 			<origin xyz="${translateX * base_x_origin_to_wheel_origin} ${translateY * base_y_origin_to_wheel_origin} ${base_z_origin_to_wheel_origin}" rpy="0 0 0" />
 			<axis xyz="0 1 0" rpy="0 0 0" />
@@ -58,8 +58,8 @@
 			<joint_properties damping="0.0" friction="0.0"/>
 		</joint>
-		<transmission name="${fb}_${lr}_wheel_tran">
+		<transmission name="${robot_ns}/${fb}_${lr}_wheel_tran">
 		  <type>transmission_interface/SimpleTransmission</type>
-		  <joint name="joint_${fb}_${lr}_wheel"/>
-		  <actuator name="${lr}_wheel_motor">
+		  <joint name="${robot_ns}/joint_${fb}_${lr}_wheel"/>
+		  <actuator name="${robot_ns}/${lr}_wheel_motor">
 		    <hardwareInterface>VelocityJointInterface</hardwareInterface>
 		    <mechanicalReduction>1</mechanicalReduction>

Commit message: Fixed some warnings from the simulator and controllers

File: aero_description/robots/aero_base.urdf.xacro (robot description, xacro)
@@ -107,4 +107,5 @@
       <topicName>imu</topicName>
       <serviceName>imu/calibrate</serviceName>
+      <gaussianNoise>0.0</gaussianNoise><!--TODO determine what this parameter is -->
     </plugin>
   </gazebo>

File: aero_description/urdf/base.urdf.xacro (robot description, xacro)
@@ -30,11 +30,4 @@
       <!-- base_footprint is a fictitious link(frame) that is on the ground right below base_link origin, navigation stack depends on this frame -->
       <link name="${robot_ns}/base_footprint">
-	<inertial>
-	  <mass value="0.0001" />
-	  <origin xyz="0 0 0" />
-	  <inertia ixx="0.0001" ixy="0.0" ixz="0.0"
-		   iyy="0.0001" iyz="0.0"
-		   izz="0.0001" />
-	</inertial>
 	<visual>
 	  <origin xyz="0 0 0" rpy="0 0 0" />

Commit message: Fliped laser in urdf to match robot

File: aero_description/robots/aero_base.urdf.xacro (robot description, xacro)
@@ -11,5 +11,5 @@
   <!-- Laser -->
   <xacro:sick_laser_v0 name="${robot_ns}/laser" parent="${robot_ns}/base_link" ros_topic="/${robot_ns}/laser" update_rate="25" >
-    <origin xyz="${base_x_size/2+0.0635} 0 0.0254" rpy="${M_PI} 0 0" />
+    <origin xyz="${base_x_size/2+0.0635} 0 0.0254" rpy="0 0 0" />
   </xacro:sick_laser_v0>
   <!-- Camera Boom -->

Commit message: Added jaco_arm to tf tree

File: aero_description/robots/aero_base.urdf.xacro (robot description, xacro)
@@ -7,4 +7,5 @@
   <xacro:include filename="$(find aero_description)/urdf/simple_transform.urdf.xacro" />
   <xacro:include filename="$(find aero_description)/urdf/camera_boom.urdf.xacro" />
+  <xacro:include filename="$(find jaco_model)/urdf/jaco_arm.xacro" />
   <property name="robot_ns" value="aero" />
   <xacro:husky robot_ns="${robot_ns}"/>
@@ -63,4 +64,52 @@
     </inertial>
   </xacro:static_transform>
+  <!-- Arm Base -->
+  <xacro:static_transform parent="aero/base_link" name="aero/arm_mount" xyz="0.3429 0 -0.023588" rpy="0 0 0">
+    <collision>
+      <origin xyz="0 0 0" rpy="0 0 0" />
+      <geometry>
+	<box size="0.01 0.01 0.01" />
+      </geometry>
+    </collision>
+    <visual>
+      <origin xyz="0 0 0" rpy="0 0 0" />
+      <geometry>
+	<box size="0.01 0.01 0.01" />
+      </geometry>
+      <material name="Blue" />
+    </visual>
+    <inertial>
+      <origin xyz="0 0 0" rpy="0 0 0"/>
+      <mass value="1"/>
+      <inertia
+	  ixx="1.0" ixy="0.0" ixz="0.0"
+	  iyy="1.0" iyz="0.0"
+	  izz="1.0"/>
+    </inertial>
+  </xacro:static_transform>
+  <xacro:static_transform parent="aero/arm_mount" name="arm_base" xyz="0 0 0" rpy="0 0 ${-M_PI/2}">
+    <collision>
+      <origin xyz="0 0 0" rpy="0 0 0" />
+      <geometry>
+	<box size="0.01 0.01 0.01" />
+      </geometry>
+    </collision>
+    <visual>
+      <origin xyz="0 0 0" rpy="0 0 0" />
+      <geometry>
+	<box size="0.01 0.01 0.01" />
+      </geometry>
+      <material name="Blue" />
+    </visual>
+    <inertial>
+      <origin xyz="0 0 0" rpy="0 0 0"/>
+      <mass value="1"/>
+      <inertia
+	  ixx="1.0" ixy="0.0" ixz="0.0"
+	  iyy="1.0" iyz="0.0"
+	  izz="1.0"/>
+    </inertial>
+  </xacro:static_transform>
+  <xacro:jaco_arm  parent="arm_base"/>
   <gazebo reference="${robot_ns}/imu">
     <sensor name="imu_sensor" type="imu"><!--from atlas-->

Commit message: Moved arm_base to fit hole in new collision box

File: aero_description/robots/aero_base.urdf.xacro (robot description, xacro)
@@ -65,5 +65,5 @@
   </xacro:static_transform>
   <!-- Arm Base -->
-  <xacro:static_transform parent="aero/base_link" name="aero/arm_mount" xyz="0.3429 0 -0.0426" rpy="0 0 0">
+  <xacro:static_transform parent="aero/base_link" name="aero/arm_mount" xyz="0.323 0 -0.0426" rpy="0 0 0">
     <collision>
       <origin xyz="0 0 0" rpy="0 0 0" />

File: aero_description/urdf/base.urdf.xacro (robot description, xacro)
@@ -64,7 +64,7 @@
 	</visual>
 	<collision>
-	  <origin xyz="0 0 0" rpy="0 0 0" />
+	  <origin xyz="-0.40 -0.203 0" rpy="${M_PI/2} 0 ${M_PI/2}" />
 	  <geometry>
-	    <mesh filename="package://aero_description/meshes/base_collision.STL" />
+            <mesh filename="package://aero_description/meshes/base_collision.STL" />
 	  </geometry>
 	  <material name="Black" />

Commit message: Flipped and move LIDAR to match robot. Disabled collision stl for LIDAR for efficiency.

File: aero_description/robots/aero_base.urdf.xacro (robot description, xacro)
@@ -12,5 +12,5 @@
   <!-- Laser -->
   <xacro:sick_laser_v0 name="${robot_ns}/laser" parent="${robot_ns}/base_link" ros_topic="/${robot_ns}/laser" update_rate="25" >
-    <origin xyz="${base_x_size/2+0.0635} 0 0.0254" rpy="0 0 0" />
+    <origin xyz="${base_x_size/2 - 0.035} 0 0.16" rpy="${M_PI} 0 0" />
   </xacro:sick_laser_v0>
   <!-- Camera Boom -->

File: aero_description/urdf/sick_laser.urdf.xacro (robot description, xacro)
@@ -21,4 +21,5 @@
         </geometry>
       </visual>
+      <!--
       <collision>
       <origin xyz="0 0 0" rpy="0 0 0" />
@@ -27,4 +28,5 @@
       </geometry>
     </collision>
+    -->
     </link>
     <!-- gazebo extensions -->
